File: Omega2/Omega2.kicad_sch (KiCad schematic)
At the start: 15 parts, among them J1 Conn_01x04_Female, J2 Conn_01x14_Female, J3 Conn_01x07_Female, SW1 SW_DIP_x01, U1 Omega2+

Commit message: edicion
Parts:
- R4: renamed from R?; value 5.1k -> (none); footprint Resistor_SMD:R_0805_2012Metric_Pad1.20x1.40mm_HandSolder -> (none)
- SW3: value (none) -> BW; footprint (none) -> TerminalBlock:TerminalBlock_Altech_AK300-2_P5.00mm
- gave numbers to parts that had none: 5
Changed lines of the file:
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@@
   (symbol (lib_id "Device:C") (at 171.45 105.41 180) (unit 1)
     (in_bom yes) (on_board yes) (fields_autoplaced)
-    (property "Reference" "C?" (id 0) (at 175.26 104.1399 0)
+    (property "Reference" "C2" (id 0) (at 175.26 104.1399 0)
       (effects (font (size 1.27 1.27)) (justify right))
     )
@@
   (symbol (lib_name "R_1") (lib_id "Device:R") (at 160.02 100.33 0) (unit 1)
     (in_bom yes) (on_board yes) (fields_autoplaced)
-    (property "Reference" "R?" (id 0) (at 162.56 99.0599 0)
+    (property "Reference" "R6" (id 0) (at 162.56 99.0599 0)
       (effects (font (size 1.27 1.27)) (justify left))
     )
@@
   (symbol (lib_id "Device:C") (at 139.7 105.41 180) (unit 1)
     (in_bom yes) (on_board yes) (fields_autoplaced)
-    (property "Reference" "C?" (id 0) (at 143.51 104.1399 0)
+    (property "Reference" "C1" (id 0) (at 143.51 104.1399 0)
       (effects (font (size 1.27 1.27)) (justify right))
     )
@@
   (symbol (lib_name "R_1") (lib_id "Device:R") (at 128.27 100.33 0) (unit 1)
     (in_bom yes) (on_board yes) (fields_autoplaced)
-    (property "Reference" "R?" (id 0) (at 130.81 99.0599 0)
-      (effects (font (size 1.27 1.27)) (justify left))
-    )
-    (property "Value" "5.1k" (id 1) (at 130.81 101.5999 0)
-      (effects (font (size 1.27 1.27)) (justify left))
-    )
-    (property "Footprint" "Resistor_SMD:R_0805_2012Metric_Pad1.20x1.40mm_HandSolder" (id 2) (at 126.492 100.33 90)
+    (property "Reference" "R4" (id 0) (at 130.81 99.0599 0)
+      (effects (font (size 1.27 1.27)) (justify left))
+    )
+    (property "Value" "" (id 1) (at 130.81 101.5999 0)
+      (effects (font (size 1.27 1.27)) (justify left))
+    )
+    (property "Footprint" "" (id 2) (at 126.492 100.33 90)
       (effects (font (size 1.27 1.27)) hide)
     )
@@
   (symbol (lib_id "Device:R") (at 128.27 87.63 180) (unit 1)
     (in_bom yes) (on_board yes)
-    (property "Reference" "R?" (id 0) (at 132.08 86.36 0))
+    (property "Reference" "R3" (id 0) (at 132.08 86.36 0))
     (property "Value" "51k" (id 1) (at 132.08 88.9 0))
     (property "Footprint" "Resistor_SMD:R_0805_2012Metric_Pad1.20x1.40mm_HandSolder" (id 2) (at 130.048 87.63 90)
@@
   (symbol (lib_id "power:GND") (at 128.27 118.11 0) (unit 1)
     (in_bom yes) (on_board yes) (fields_autoplaced)
-    (property "Reference" "#PWR?" (id 0) (at 128.27 124.46 0)
+    (property "Reference" "#PWR0101" (id 0) (at 128.27 124.46 0)
       (effects (font (size 1.27 1.27)) hide)
     )
@@
   (symbol (lib_id "Device:R") (at 160.02 87.63 180) (unit 1)
     (in_bom yes) (on_board yes)
-    (property "Reference" "R?" (id 0) (at 163.83 86.36 0))
+    (property "Reference" "R5" (id 0) (at 163.83 86.36 0))
     (property "Value" "51k" (id 1) (at 163.83 88.9 0))
     (property "Footprint" "Resistor_SMD:R_0805_2012Metric_Pad1.20x1.40mm_HandSolder" (id 2) (at 161.798 87.63 90)
@@
       (effects (font (size 1.27 1.27)) (justify left))
     )
-    (property "Value" "" (id 1) (at 132.08 111.7599 90)
-      (effects (font (size 1.27 1.27)) (justify left))
-    )
-    (property "Footprint" "" (id 2) (at 133.35 110.49 0)
+    (property "Value" "BW" (id 1) (at 132.08 111.7599 90)
+      (effects (font (size 1.27 1.27)) (justify left))
+    )
+    (property "Footprint" "TerminalBlock:TerminalBlock_Altech_AK300-2_P5.00mm" (id 2) (at 133.35 110.49 0)
       (effects (font (size 1.27 1.27)) hide)
     )
@@
   (symbol (lib_id "power:GND") (at 160.02 118.11 0) (unit 1)
     (in_bom yes) (on_board yes) (fields_autoplaced)
-    (property "Reference" "#PWR?" (id 0) (at 160.02 124.46 0)
+    (property "Reference" "#PWR0104" (id 0) (at 160.02 124.46 0)
       (effects (font (size 1.27 1.27)) hide)
     )
@@
   )
   (symbol_instances
+    (path "/dd472471-f193-48d5-889c-efd694d3f702"
+      (reference "#PWR0101") (unit 1) (value "GND") (footprint "")
+    )
     (path "/cf7b28ee-b304-4d98-a7d3-b9234279b9f3"
       (reference "#PWR0102") (unit 1) (value "GND") (footprint "")
@@
       (reference "#PWR0103") (unit 1) (value "+3.3V") (footprint "")
     )
-    (path "/dd472471-f193-48d5-889c-efd694d3f702"
-      (reference "#PWR?") (unit 1) (value "GND") (footprint "")
-    )
     (path "/f4648014-6a49-47fe-aa14-831ac44193be"
-      (reference "#PWR?") (unit 1) (value "GND") (footprint "")
+      (reference "#PWR0104") (unit 1) (value "GND") (footprint "")
+    )
+    (path "/917dba0e-1b1e-4fc1-b97b-7105df526305"
+      (reference "C1") (unit 1) (value "100n") (footprint "Capacitor_SMD:C_0805_2012Metric_Pad1.18x1.45mm_HandSolder")
     )
     (path "/291cc86e-d7a1-4f14-983b-0e47c854bfea"
-      (reference "C?") (unit 1) (value "100n") (footprint "Capacitor_SMD:C_0805_2012Metric_Pad1.18x1.45mm_HandSolder")
-    )
-    (path "/917dba0e-1b1e-4fc1-b97b-7105df526305"
-      (reference "C?") (unit 1) (value "100n") (footprint "Capacitor_SMD:C_0805_2012Metric_Pad1.18x1.45mm_HandSolder")
+      (reference "C2") (unit 1) (value "100n") (footprint "Capacitor_SMD:C_0805_2012Metric_Pad1.18x1.45mm_HandSolder")
     )
     (path "/f52d322d-fe19-4531-ac42-28ccced54df0"
@@
       (reference "R2") (unit 1) (value "3K2") (footprint "Resistor_THT:R_Axial_DIN0204_L3.6mm_D1.6mm_P7.62mm_Horizontal")
     )
+    (path "/9c476165-300e-4e08-a354-4288b203c377"
+      (reference "R3") (unit 1) (value "51k") (footprint "Resistor_SMD:R_0805_2012Metric_Pad1.20x1.40mm_HandSolder")
+    )
+    (path "/9a0f5593-2efd-4f52-bc76-f583ab6c95eb"
+      (reference "R4") (unit 1) (value "5.1k") (footprint "Resistor_SMD:R_0805_2012Metric_Pad1.20x1.40mm_HandSolder")
+    )
+    (path "/ee19a334-b72e-4d54-9a8e-a742ee56e7f1"
+      (reference "R5") (unit 1) (value "51k") (footprint "Resistor_SMD:R_0805_2012Metric_Pad1.20x1.40mm_HandSolder")
+    )
     (path "/552d2777-af2b-41ec-a31e-cd43b7c8490e"
-      (reference "R?") (unit 1) (value "5.1k") (footprint "Resistor_SMD:R_0805_2012Metric_Pad1.20x1.40mm_HandSolder")
-    )
-    (path "/9a0f5593-2efd-4f52-bc76-f583ab6c95eb"
-      (reference "R?") (unit 1) (value "5.1k") (footprint "Resistor_SMD:R_0805_2012Metric_Pad1.20x1.40mm_HandSolder")
-    )
-    (path "/9c476165-300e-4e08-a354-4288b203c377"
-      (reference "R?") (unit 1) (value "51k") (footprint "Resistor_SMD:R_0805_2012Metric_Pad1.20x1.40mm_HandSolder")
-    )
-    (path "/ee19a334-b72e-4d54-9a8e-a742ee56e7f1"
-      (reference "R?") (unit 1) (value "51k") (footprint "Resistor_SMD:R_0805_2012Metric_Pad1.20x1.40mm_HandSolder")
+      (reference "R6") (unit 1) (value "5.1k") (footprint "Resistor_SMD:R_0805_2012Metric_Pad1.20x1.40mm_HandSolder")
     )
     (path "/efe02569-b4d6-46d8-a69d-741dd0f4d887"

Commit message: edicion pcb
Parts:
- R4: value (none) -> 5.1k; footprint (none) -> Resistor_SMD:R_0805_2012Metric_Pad1.20x1.40mm_HandSolder
- SW2: value (none) -> FW; footprint (none) -> TerminalBlock:TerminalBlock_Altech_AK300-2_P5.00mm
Changed lines of the file:
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@@
       (effects (font (size 1.27 1.27)) (justify left))
     )
-    (property "Value" "" (id 1) (at 163.83 111.7599 90)
+    (property "Value" "FW" (id 1) (at 163.83 111.7599 90)
       (effects (font (size 1.27 1.27)) (justify left))
     )
-    (property "Footprint" "" (id 2) (at 165.1 110.49 0)
+    (property "Footprint" "TerminalBlock:TerminalBlock_Altech_AK300-2_P5.00mm" (id 2) (at 165.1 110.49 0)
       (effects (font (size 1.27 1.27)) hide)
     )
@@
       (effects (font (size 1.27 1.27)) (justify left))
     )
-    (property "Value" "" (id 1) (at 130.81 101.5999 0)
+    (property "Value" "5.1k" (id 1) (at 130.81 101.5999 0)
       (effects (font (size 1.27 1.27)) (justify left))
     )
-    (property "Footprint" "" (id 2) (at 126.492 100.33 90)
+    (property "Footprint" "Resistor_SMD:R_0805_2012Metric_Pad1.20x1.40mm_HandSolder" (id 2) (at 126.492 100.33 90)
       (effects (font (size 1.27 1.27)) hide)
     )

Commit message: union de todo en el mismo esquemático
Parts:
- added C1, C2, C4, C5: (no value), symbol Adafruit MAX98357 Breakout-eagle-import:CAP_CERAMIC0805-NOOUTLINE
- added FB1, FB2: (no value), symbol Adafruit MAX98357 Breakout-eagle-import:FERRITE-0805NO
- added FID1, FID2: (no value), symbol Adafruit MAX98357 Breakout-eagle-import:FIDUCIAL{dblquote}{dblquote}
- added JP1: (no value), symbol Adafruit MAX98357 Breakout-eagle-import:HEADER-1X7THICKER
- added R1: (no value), symbol Adafruit MAX98357 Breakout-eagle-import:RESISTOR0805_NOOUTLINE
- added U$10, U$9: (no value), symbol Adafruit MAX98357 Breakout-eagle-import:MOUNTINGHOLE2.5
- added U1: (no value), symbol Adafruit MAX98357 Breakout-eagle-import:AUDIOAMP_MAX98357
- added X1: (no value), symbol Adafruit MAX98357 Breakout-eagle-import:TERMBLOCK_1X2
Connections:
- net GND: now also C1.2, C2.2, C4.2, C5.2, JP1.2, U1.11 (GND), U1.15 (GND), U1.3 (GND), U1.THERMAL (GND)
- new net: FB1.1 (P$1), U1.9 (OUTP)
- new net: FB2.1 (P$1), U1.10 (OUTN)
- new net BCLK: JP1.6, U1.16 (BCLK)
- new net DIN: JP1.5, U1.1 (DIN)
- new net GAIN: JP1.4, U1.2 (GAIN)
- new net LRCLK: JP1.7, U1.14 (LRCLK)
- new net SD_MODE: JP1.3, R1.1, U1.4 (~{SD_MODE})
- new net VDD: C1.1, C2.1, JP1.1, R1.2, U1.7 (VDD), U1.8 (VDD)
- new net VO+: C5.1, FB1.2 (P$2), X1.2
- new net VO-: C4.1, FB2.2 (P$2), X1.1
Other:
- note added: "Gain=9dB"
- note added: "R1 Channel Selection: LEFT = VDD (0 Ohm) RIGHT = 370K (94*VDD-100) LEFT/2 + RIGHT/2 = 1.011M (222.2*VDD-100)"
- note added: "ToDo: Ferrite (select w/high Z at high F, low Z at low F). Try to block everything >1MHz or so."
- moved on the sheet: C1, C2, J3, R3, R4, R5, R6, SW2, SW3

Commit message: esquemático editado
Parts:
- C1, C2, C4, C5, FB1, FB2, FID1, FID2, JP1, R1, U$10, U$9, U1, X1: value (none) -> ~
Connections:
- net LRCLK is gone; now on net Om2: JP1.7, U1.14 (LRCLK)
- net +3V3: now also C1.1, C2.1, JP1.1, U1.7 (VDD), U1.8 (VDD)
- removed net VDD: C1.1, C2.1, JP1.1, R1.2, U1.7 (VDD), U1.8 (VDD)
