File: etapa_potencia/REEL/REEL/REEL.kicad_sch (KiCad schematic)
At the start: 30 parts, among them J1 USB_B_Mini, SW1 SW_Push, SW2 SW_Reed, SW3 SW_Push, U1 Tp5400, U2 ESP32-WROOM-32, U3 FT232, U4 AMS1117-3.3

Commit message: Display
Parts:
- removed BT1: Battery_Cell, Battery:BatteryHolder_Bulgin_BX0036_1xC, symbol Device:Battery_Cell
- removed C10, C2, C9: 10u, Capacitor_SMD:C_1210_3225Metric_Pad1.33x2.70mm_HandSolder, symbol Device:C
- removed C3, C5: 0.1u, Capacitor_SMD:C_0603_1608Metric_Pad1.08x0.95mm_HandSolder, symbol Device:C
- removed C4, C6: 22u, Capacitor_SMD:C_1210_3225Metric_Pad1.33x2.70mm_HandSolder, symbol Device:C
- removed C7: 47u, Capacitor_SMD:C_1210_3225Metric_Pad1.33x2.70mm_HandSolder, symbol Device:C
- removed D1: Green, LED_SMD:LED_0805_2012Metric_Pad1.15x1.40mm_HandSolder, symbol Device:LED
- removed D2: Red, LED_SMD:LED_0805_2012Metric_Pad1.15x1.40mm_HandSolder, symbol Device:LED
- removed D3: SMBJ5383B, SMBJ5383B:SMBJ5383B, symbol Device:D_Schottky
- removed J1: USB_B_Mini, Connector_USB:USB_Mini-B_AdamTech_MUSB-B5-S-VT-TSMT-1_SMD_Vertical, symbol Connector:USB_B_Mini
- removed L1: 10u, Inductor_SMD:L_0805_2012Metric_Pad1.05x1.20mm_HandSolder, symbol Device:L
- removed R1: 1k, Resistor_SMD:R_1218_3246Metric_Pad1.22x4.75mm_HandSolder, symbol Device:R
- removed R3, R4: 1, Resistor_SMD:R_1218_3246Metric_Pad1.22x4.75mm_HandSolder, symbol Device:R
- removed R5: 1.1k, Resistor_SMD:R_1218_3246Metric_Pad1.22x4.75mm_HandSolder, symbol Device:R
- removed U1: Tp5400, symbol TP5400:Tp5400
- removed U4: AMS1117-3.3, Package_TO_SOT_SMD:SOT-223-3_TabPin2, symbol Regulator_Linear:AMS1117-3.3
- added C? (x2): 100n, Capacitor_SMD:C_0805_2012Metric_Pad1.18x1.45mm_HandSolder, symbol Device:C
- added J?: Conn_01x14_Female, Connector_PinSocket_2.54mm:PinSocket_1x14_P2.54mm_Vertical, symbol Connector:Conn_01x14_Female
- added J?: Conn_01x07_Female, Connector_PinSocket_2.54mm:PinSocket_1x07_P2.54mm_Vertical, symbol Connector:Conn_01x07_Female
- added J?: Conn_01x04_Female, Connector_PinSocket_2.54mm:PinSocket_1x04_P2.54mm_Vertical, symbol Connector:Conn_01x04_Female
- added R? (x2): 51k, Resistor_SMD:R_0805_2012Metric_Pad1.20x1.40mm_HandSolder, symbol Device:R
- added R? (x2): 5.1k, Resistor_SMD:R_0805_2012Metric_Pad1.20x1.40mm_HandSolder, symbol Device:R
- added SW?: BW, TerminalBlock:TerminalBlock_Altech_AK300-2_P5.00mm, symbol Switch:SW_Push
- added SW?: FW, TerminalBlock:TerminalBlock_Altech_AK300-2_P5.00mm, symbol Switch:SW_Push
Connections:
- net +3V3: now also J?.14 (Pin_14), J?.7 (Pin_7)
- net GND: now also C?.1, C?.1, J?.13 (Pin_13), SW?.2, SW?.2
- net CS: now reaches U2.23 (IO15)
- net CS: now also J?.12 (Pin_12)
- net SCK: now reaches U2.30 (IO18)
- net SCK: now also J?.8 (Pin_8)
- net MOSI: now reaches U2.37 (IO23)
- net MOSI: now also J?.9 (Pin_9)
- net Rst_d: now reaches U2.6 (IO34)
- net Rst_d: now also J?.11 (Pin_11)
- net D/C: now reaches U2.7 (IO35)
- net D/C: now also J?.10 (Pin_10)
- net GPIO0 renamed IO0
- net RESET renamed EN
- new net: R?.2, SW?.1 (x2)
- new net 3.3V: R?.2, R?.2
- new net Om11: J?.3 (Pin_3)
- new net Om12: J?.4 (Pin_4)
- new net Om13: J?.5 (Pin_5)
- new net Om16: C?.2, R?.1, R?.1
- new net Om17: C?.2, R?.1, R?.1
- new net Om18: J?.6 (Pin_6)
- new net Om19: J?.7 (Pin_7)
- new net Om4: J?.1 (Pin_1)
- new net Om5: J?.2 (Pin_2)
- no-connect marks 32 -> 26
Other:
- added sheet Power (power.kicad_sch)
- note added: "Botones"
- note added: "Circuito de programación"
- note added: "Display"
- note added: "Programador"
- note added: "Reset"
- note added: "Teclado"
- note removed: "Cargador"
- note removed: "Regulador"
- moved on the sheet: C1, C8, R2, R6, R7, SW1, SW3, U3

Commit message: Adición etapa de audio
Parts:
- added J?: Conn_01x07_Female, Connector_PinSocket_2.54mm:PinSocket_1x07_P2.54mm_Vertical, symbol Connector:Conn_01x07_Female
Connections:
- net +3V3: now also J?.1 (Pin_1)
- net GND: now also J?.2 (Pin_2)
- net I2S_DIN: now reaches U2.14 (IO12)
- net I2S_DIN: now also J?.5 (Pin_5)
- net I2S_WS: now reaches U2.26 (IO4)
- net I2S_WS: now also J?.7 (Pin_7)
- net I2S_CLK: now reaches U2.29 (IO5)
- net I2S_CLK: now also J?.6 (Pin_6)
- no-connect marks 26 -> 28
Other:
- note added: "Audio"
Changed lines of the file:
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@@
   (no_connect (at 124.46 119.38))
   (no_connect (at 93.98 149.86))
+  (no_connect (at 228.6 54.61))
   (no_connect (at 93.98 121.92))
   (no_connect (at 124.46 157.48))
@@
   (no_connect (at 124.46 124.46))
   (no_connect (at 124.46 167.64))
+  (no_connect (at 228.6 57.15))
   (no_connect (at 124.46 149.86))
   (no_connect (at 124.46 162.56))
@@
     (stroke (width 0) (type default) (color 0 0 0 0))
   )
+  (polyline (pts (xy 207.01 69.85) (xy 207.01 41.91))
+    (stroke (width 0) (type default) (color 0 0 0 0))
+  )
+  (wire (pts (xy 127 124.46) (xy 124.46 124.46))
+    (stroke (width 0) (type default) (color 0 0 0 0))
+  )
   (polyline (pts (xy 66.04 142.24) (xy 66.04 190.5))
     (stroke (width 0) (type default) (color 0 0 0 0))
@@
     (stroke (width 0) (type default) (color 0 0 0 0))
   )
+  (wire (pts (xy 226.06 64.77) (xy 228.6 64.77))
+    (stroke (width 0) (type default) (color 0 0 0 0))
+  )
   (wire (pts (xy 93.98 46.99) (xy 93.98 49.53))
     (stroke (width 0) (type default) (color 0 0 0 0))
@@
     (stroke (width 0) (type default) (color 0 0 0 0))
   )
+  (wire (pts (xy 226.06 57.15) (xy 228.6 57.15))
+    (stroke (width 0) (type default) (color 0 0 0 0))
+  )
   (wire (pts (xy 125.73 57.15) (xy 125.73 58.42))
     (stroke (width 0) (type default) (color 0 0 0 0))
   )
+  (wire (pts (xy 226.06 49.53) (xy 234.95 49.53))
+    (stroke (width 0) (type default) (color 0 0 0 0))
+  )
   (wire (pts (xy 57.15 53.34) (xy 58.42 53.34))
     (stroke (width 0) (type default) (color 0 0 0 0))
@@
     (stroke (width 0) (type default) (color 0 0 0 0))
   )
+  (wire (pts (xy 226.06 62.23) (xy 228.6 62.23))
+    (stroke (width 0) (type default) (color 0 0 0 0))
+  )
   (wire (pts (xy 257.81 135.89) (xy 252.73 135.89))
     (stroke (width 0) (type default) (color 0 0 0 0))
@@
     (stroke (width 0) (type default) (color 0 0 0 0))
   )
+  (wire (pts (xy 226.06 54.61) (xy 228.6 54.61))
+    (stroke (width 0) (type default) (color 0 0 0 0))
+  )
   (wire (pts (xy 54.61 167.64) (xy 57.15 167.64))
     (stroke (width 0) (type default) (color 0 0 0 0))
@@
     (stroke (width 0) (type default) (color 0 0 0 0))
   )
-  (wire (pts (xy 109.22 180.34) (xy 109.22 184.15))
+  (wire (pts (xy 109.22 180.34) (xy 109.22 182.88))
+    (stroke (width 0) (type default) (color 0 0 0 0))
+  )
+  (polyline (pts (xy 241.3 41.91) (xy 241.3 69.85))
     (stroke (width 0) (type default) (color 0 0 0 0))
   )
@@
     (stroke (width 0) (type default) (color 0 0 0 0))
   )
+  (wire (pts (xy 226.06 59.69) (xy 228.6 59.69))
+    (stroke (width 0) (type default) (color 0 0 0 0))
+  )
   (wire (pts (xy 44.45 128.27) (xy 48.26 128.27))
     (stroke (width 0) (type default) (color 0 0 0 0))
@@
     (stroke (width 0) (type default) (color 0 0 0 0))
   )
+  (wire (pts (xy 226.06 52.07) (xy 234.95 52.07))
+    (stroke (width 0) (type default) (color 0 0 0 0))
+  )
   (wire (pts (xy 252.73 133.35) (xy 251.46 133.35))
     (stroke (width 0) (type default) (color 0 0 0 0))
   )
+  (wire (pts (xy 127 127) (xy 124.46 127))
+    (stroke (width 0) (type default) (color 0 0 0 0))
+  )
   (wire (pts (xy 210.82 130.81) (xy 223.52 130.81))
     (stroke (width 0) (type default) (color 0 0 0 0))
@@
     (stroke (width 0) (type default) (color 0 0 0 0))
   )
+  (polyline (pts (xy 207.01 41.91) (xy 241.3 41.91))
+    (stroke (width 0) (type default) (color 0 0 0 0))
+  )
   (wire (pts (xy 167.64 62.23) (xy 170.18 62.23))
     (stroke (width 0) (type default) (color 0 0 0 0))
@@
     (stroke (width 0) (type default) (color 0 0 0 0))
   )
+  (polyline (pts (xy 241.3 69.85) (xy 207.01 69.85))
+    (stroke (width 0) (type default) (color 0 0 0 0))
+  )
   (polyline (pts (xy 280.67 151.13) (xy 280.67 120.65))
     (stroke (width 0) (type default) (color 0 0 0 0))
@@
   )
   (wire (pts (xy 48.26 114.3) (xy 48.26 116.84))
+    (stroke (width 0) (type default) (color 0 0 0 0))
+  )
+  (wire (pts (xy 127 129.54) (xy 124.46 129.54))
     (stroke (width 0) (type default) (color 0 0 0 0))
   )
@@
     (effects (font (size 1.27 1.27) (thickness 0.254) bold) (justify left bottom))
   )
+  (text "Audio" (at 208.28 68.58 0)
+    (effects (font (size 1.27 1.27)) (justify left bottom))
+  )
   (text "Programador" (at 242.57 124.46 0)
     (effects (font (size 1.27 1.27) (thickness 0.254) bold) (justify left bottom))
@@
     (effects (font (size 1.27 1.27)) (justify left bottom))
   )
+  (label "I2S_CLK" (at 228.6 62.23 0)
+    (effects (font (size 1.27 1.27)) (justify left bottom))
+  )
+  (label "I2S_DIN" (at 228.6 59.69 0)
+    (effects (font (size 1.27 1.27)) (justify left bottom))
+  )
   (label "SCK" (at 127 144.78 0)
     (effects (font (size 1.27 1.27)) (justify left bottom))
@@
     (effects (font (size 1.27 1.27)) (justify right bottom))
   )
+  (label "I2S_CLK" (at 127 127 0)
+    (effects (font (size 1.27 1.27)) (justify left bottom))
+  )
   (label "IO0" (at 194.31 143.51 180)
     (effects (font (size 1.27 1.27)) (justify right bottom))
@@
     (effects (font (size 1.27 1.27)) (justify left bottom))
   )
+  (label "I2S_DIN" (at 127 129.54 0)
+    (effects (font (size 1.27 1.27)) (justify left bottom))
+  )
   (label "MOSI" (at 58.42 53.34 0)
     (effects (font (size 1.27 1.27)) (justify left bottom))
   )
   (label "D{slash}C" (at 58.42 55.88 0)
+    (effects (font (size 1.27 1.27)) (justify left bottom))
+  )
+  (label "I2S_WS" (at 127 124.46 0)
     (effects (font (size 1.27 1.27)) (justify left bottom))
   )
@@
   )
   (label "CS" (at 127 137.16 0)
+    (effects (font (size 1.27 1.27)) (justify left bottom))
+  )
+  (label "I2S_WS" (at 228.6 64.77 0)
     (effects (font (size 1.27 1.27)) (justify left bottom))
   )
@@
     (pin "1")
     (pin "2")
+  )
+  (symbol (lib_id "power:GND") (at 234.95 52.07 90) (unit 1)
+    (in_bom yes) (on_board yes)
+    (property "Reference" "#PWR?" (id 0) (at 241.3 52.07 0)
+      (effects (font (size 1.27 1.27)) hide)
+    )
+    (property "Value" "GND" (id 1) (at 239.3442 51.943 0))
+    (property "Footprint" "" (id 2) (at 234.95 52.07 0)
+      (effects (font (size 1.27 1.27)) hide)
+    )
+    (property "Datasheet" "" (id 3) (at 234.95 52.07 0)
+      (effects (font (size 1.27 1.27)) hide)
+    )
+    (pin "1")
   )
   (symbol (lib_id "power:GND") (at 66.04 63.5 0) (unit 1)
@@
     (pin "1")
   )
-  (symbol (lib_id "power:GND") (at 109.22 184.15 0) (unit 1)
-    (in_bom yes) (on_board yes)
-    (property "Reference" "#PWR09" (id 0) (at 109.22 190.5 0)
-      (effects (font (size 1.27 1.27)) hide)
-    )
-    (property "Value" "GND" (id 1) (at 109.347 188.5442 0))
-    (property "Footprint" "" (id 2) (at 109.22 184.15 0)
-      (effects (font (size 1.27 1.27)) hide)
-    )
-    (property "Datasheet" "" (id 3) (at 109.22 184.15 0)
+  (symbol (lib_id "Connector:Conn_01x07_Female") (at 220.98 57.15 0) (mirror y) (unit 1)
+    (in_bom yes) (on_board yes)
+    (property "Reference" "J?" (id 0) (at 224.79 43.18 0)
+      (effects (font (size 1.27 1.27)) (justify left))
+    )
+    (property "Value" "Conn_01x07_Female" (id 1) (at 228.6 45.72 0)
+      (effects (font (size 1.27 1.27)) (justify left))
+    )
+    (property "Footprint" "Connector_PinSocket_2.54mm:PinSocket_1x07_P2.54mm_Vertical" (id 2) (at 220.98 57.15 0)
+      (effects (font (size 1.27 1.27)) hide)
+    )
+    (property "Datasheet" "~" (id 3) (at 220.98 57.15 0)
+      (effects (font (size 1.27 1.27)) hide)
+    )
+    (pin "1")
+    (pin "2")
+    (pin "3")
+    (pin "4")
+    (pin "5")
+    (pin "6")
+    (pin "7")
+  )
+  (symbol (lib_id "power:GND") (at 109.22 182.88 0) (unit 1)
+    (in_bom yes) (on_board yes)
+    (property "Reference" "#PWR09" (id 0) (at 109.22 189.23 0)
+      (effects (font (size 1.27 1.27)) hide)
+    )
+    (property "Value" "GND" (id 1) (at 109.347 187.2742 0))
+    (property "Footprint" "" (id 2) (at 109.22 182.88 0)
+      (effects (font (size 1.27 1.27)) hide)
+    )
+    (property "Datasheet" "" (id 3) (at 109.22 182.88 0)
       (effects (font (size 1.27 1.27)) hide)
     )
@@
     (pin "2")
   )
+  (symbol (lib_id "power:+3.3V") (at 234.95 49.53 0) (unit 1)
+    (in_bom yes) (on_board yes)
+    (property "Reference" "#PWR?" (id 0) (at 234.95 53.34 0)
+      (effects (font (size 1.27 1.27)) hide)
+    )
+    (property "Value" "+3.3V" (id 1) (at 235.331 45.1358 0))
+    (property "Footprint" "" (id 2) (at 234.95 49.53 0)
+      (effects (font (size 1.27 1.27)) hide)
+    )
+    (property "Datasheet" "" (id 3) (at 234.95 49.53 0)
+      (effects (font (size 1.27 1.27)) hide)
+    )
+    (pin "1")
+  )
   (sheet (at 25.4 113.03) (size 19.05 17.78) (fields_autoplaced)
     (stroke (width 0.1524) (type solid) (color 0 0 0 0))
@@
       (reference "#PWR?") (unit 1) (value "GND") (footprint "")
     )
+    (path "/40afe74c-181d-4dc9-b4fa-6dc9efc48174"
+      (reference "#PWR?") (unit 1) (value "GND") (footprint "")
+    )
     (path "/4a4fbfc3-3481-48e6-b7c9-21e9a9ace57c"
       (reference "#PWR?") (unit 1) (value "GND") (footprint "")
@@
       (reference "#PWR?") (unit 1) (value "+5V") (footprint "")
     )
+    (path "/fc9ee4bb-f75d-4734-a7b9-19682b58dabb"
+      (reference "#PWR?") (unit 1) (value "+3.3V") (footprint "")
+    )
     (path "/05689d2f-cd22-43d5-af77-23d23536e452/a15da288-795e-497a-8e6b-e8012bc97551"
       (reference "BT1") (unit 1) (value "Battery_Cell") (footprint "Battery:BatteryHolder_Bulgin_BX0036_1xC")
@@
       (reference "J?") (unit 1) (value "Conn_01x14_Female") (footprint "Connector_PinSocket_2.54mm:PinSocket_1x14_P2.54mm_Vertical")
     )
+    (path "/95c67197-60ac-4483-839b-3e7f5dc412a8"
+      (reference "J?") (unit 1) (value "Conn_01x07_Female") (footprint "Connector_PinSocket_2.54mm:PinSocket_1x07_P2.54mm_Vertical")
+    )
     (path "/a92e3d47-777a-42a3-a090-079534c88be0"
