File: etapa_potencia/REEL/REEL/REEL.kicad_sch (KiCad schematic)
At the start: 24 parts, among them J1 Conn_display2, J2 Conn_display_2, J3 Conn_teclado, J4 Conn_audio, J6 Salida_amp, J7 Entrada_buzzer, SW1 SW_Push, SW3 SW_Push, SW4 BW, SW5 FW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

Commit message: Ordenar huellas en PCB ahora sí
Parts:
- R6: footprint (none) -> Resistor_SMD:R_0805_2012Metric_Pad1.20x1.40mm_HandSolder
- SW1: footprint (none) -> Button_Switch_SMD:SW_SPST_CK_RS282G05A3
Connections:
- net FW: now also U2.14 (IO12); no longer U2.37 (IO23)
- net SDMISO: now also U2.12 (IO27); no longer U2.33 (IO21)
- net T1: now also U2.37 (IO23); no longer U2.36 (IO22)
- net T2: now also U2.36 (IO22); no longer U2.12 (IO27)
- net T3: now also U2.33 (IO21); no longer U2.14 (IO12)
Changed lines of the file:
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@@
-    (stroke (width 0) (type default) (color 0 0 0 0))
-  )
-  (wire (pts (xy 129.54 148.59) (xy 133.35 148.59))
     (stroke (width 0) (type default) (color 0 0 0 0))
   )
@@
     (stroke (width 0) (type default) (color 0 0 0 0))
   )
+  (wire (pts (xy 133.35 143.51) (xy 129.54 143.51))
+    (stroke (width 0) (type default) (color 0 0 0 0))
+  )
   (wire (pts (xy 137.16 62.23) (xy 137.16 69.85))
     (stroke (width 0) (type default) (color 0 0 0 0))
@@
     (stroke (width 0) (type default) (color 0 0 0 0))
   )
-  (wire (pts (xy 132.08 146.05) (xy 129.54 146.05))
-    (stroke (width 0) (type default) (color 0 0 0 0))
-  )
   (wire (pts (xy 62.23 161.29) (xy 64.77 161.29))
     (stroke (width 0) (type default) (color 0 0 0 0))
@@
     (stroke (width 0) (type default) (color 0 0 0 0))
   )
+  (wire (pts (xy 133.35 148.59) (xy 129.54 148.59))
+    (stroke (width 0) (type default) (color 0 0 0 0))
+  )
   (wire (pts (xy 52.07 57.15) (xy 60.96 57.15))
     (stroke (width 0) (type default) (color 0 0 0 0))
@@
     (stroke (width 0) (type default) (color 0 0 0 0))
   )
-  (wire (pts (xy 132.08 123.19) (xy 129.54 123.19))
-    (stroke (width 0) (type default) (color 0 0 0 0))
-  )
   (wire (pts (xy 125.73 68.58) (xy 125.73 69.85))
     (stroke (width 0) (type default) (color 0 0 0 0))
@@
     (stroke (width 0) (type default) (color 0 0 0 0))
   )
-  (wire (pts (xy 129.54 156.21) (xy 133.35 156.21))
+  (wire (pts (xy 130.81 156.21) (xy 129.54 156.21))
     (stroke (width 0) (type default) (color 0 0 0 0))
   )
@@
     (stroke (width 0) (type default) (color 0 0 0 0))
   )
+  (wire (pts (xy 133.35 146.05) (xy 129.54 146.05))
+    (stroke (width 0) (type default) (color 0 0 0 0))
+  )
   (polyline (pts (xy 200.66 26.67) (xy 247.65 26.67))
     (stroke (width 0) (type default) (color 0 0 0 0))
@@
     (stroke (width 0) (type default) (color 0 0 0 0))
   )
+  (wire (pts (xy 133.35 123.19) (xy 129.54 123.19))
+    (stroke (width 0) (type default) (color 0 0 0 0))
+  )
   (polyline (pts (xy 247.65 54.61) (xy 200.66 54.61))
     (stroke (width 0) (type default) (color 0 0 0 0))
@@
   )
   (wire (pts (xy 93.98 69.85) (xy 105.41 69.85))
-    (stroke (width 0) (type default) (color 0 0 0 0))
-  )
-  (wire (pts (xy 129.54 143.51) (xy 132.08 143.51))
     (stroke (width 0) (type default) (color 0 0 0 0))
   )
@@
     (effects (font (size 1.27 1.27)) (justify left bottom))
   )
-  (label "T2" (at 133.35 156.21 0)
+  (label "T2" (at 133.35 146.05 0)
     (effects (font (size 1.27 1.27)) (justify left bottom))
   )
@@
     (effects (font (size 1.27 1.27)) (justify left bottom))
   )
-  (label "T1" (at 132.08 146.05 0)
+  (label "T1" (at 133.35 148.59 0)
     (effects (font (size 1.27 1.27)) (justify left bottom))
   )
@@
     (effects (font (size 1.27 1.27)) (justify left bottom))
   )
-  (label "SDMISO" (at 132.08 143.51 0)
+  (label "SDMISO" (at 130.81 156.21 0)
     (effects (font (size 1.27 1.27)) (justify left bottom))
   )
@@
     (effects (font (size 1.27 1.27)) (justify left bottom))
   )
-  (label "T3" (at 132.08 123.19 0)
+  (label "T3" (at 133.35 143.51 0)
     (effects (font (size 1.27 1.27)) (justify left bottom))
   )
@@
     (effects (font (size 1.27 1.27)) (justify left bottom))
   )
-  (label "FW" (at 133.35 148.59 0)
+  (label "FW" (at 133.35 123.19 0)
     (effects (font (size 1.27 1.27)) (justify left bottom))
   )
@@
       (effects (font (size 1.27 1.27)) (justify left))
     )
-    (property "Footprint" "" (id 2) (at 189.23 132.588 90)
+    (property "Footprint" "Resistor_SMD:R_0805_2012Metric_Pad1.20x1.40mm_HandSolder" (id 2) (at 189.23 132.588 90)
       (effects (font (size 1.27 1.27)) hide)
     )
@@
       (effects (font (size 1.27 1.27)) (justify right))
     )
-    (property "Footprint" "" (id 2) (at 57.15 170.18 0)
-      (effects (font (size 1.27 1.27)) hide)
-    )
+    (property "Footprint" "Button_Switch_SMD:SW_SPST_CK_RS282G05A3" (id 2) (at 57.15 170.18 0)
+      (effects (font (size 1.27 1.27)) hide)
+    )
